Commit message: feat: port from Humble/Gazebo Classic to Jazzy/Gazebo Harmonic
- Replace gazebo_ros with ros_gz_sim and ros_gz_bridge
- Update URDF plugins: libgazebo_ros_diff_drive -> gz-sim-diff-drive-system,
  libgazebo_ros_camera -> native Gazebo Harmonic sensor
- Add ros_gz_bridge for cmd_vel, odom, camera, tf topic bridging
- Strip embedded robot model from world files (spawn from URDF instead)
- Use robot_description parameter instead of URDF file argument

File: path_planning_ws/src/maze_bot/urdf/maze_bot.urdf (robot description, URDF)
Before this commit: robot maze_bot, 6 links, 5 joints
Joints:
- joint wheel_right_joint: origin xyz=0.09 0.085 0.04   rpy=0 0.0 0.0 -> xyz=0.09 0.085 0.04 rpy=0 0.0 0.0
